Commit message: Added a laser scan sensor

File: m2wr_description/urdf/m2wr.xacro (robot description, xacro)
@@ -49,4 +49,29 @@
     </visual>
   </link>
+  <link name="sensor_laser">
+    <inertial>
+        <origin xyz="0 0 0" rpy="0 0 0" />
+        <mass value="1" />
+        <xacro:cylinder_inertia mass="1" r="0.05" l="0.1" />
+    </inertial>
+    <visual>
+        <origin xyz="0 0 0" rpy="0 0 0" />
+        <geometry>
+        <cylinder radius="0.05" length="0.1"/>
+        </geometry>
+        <material name="white" />
+    </visual>
+    <collision>
+        <origin xyz="0 0 0" rpy="0 0 0"/>
+        <geometry>
+        <cylinder radius="0.05" length="0.1"/>
+        </geometry>
+    </collision>
+  </link>
+  <joint name="joint_sensor_laser" type="fixed">
+    <origin xyz="0.15 0 0.05" rpy="0 0 0"/>
+    <parent link="link_chassis"/>
+    <child link="sensor_laser"/>
+  </joint>
   <xacro:link_wheel name="link_left_wheel" />
   <xacro:joint_wheel name="joint_left_wheel" child="link_left_wheel" origin="-0.05 -0.15 0"/>

File: m2wr_description/urdf/macros.xacro (robot description, xacro)
@@ -32,3 +32,8 @@
         </joint>
     </macro>
+    <macro name="cylinder_inertia" params="mass r l">
+        <inertia  ixx="${mass*(3*r*r+l*l)/12}" ixy = "0" ixz = "0"
+                    iyy="${mass*(3*r*r+l*l)/12}" iyz = "0"
+                    izz="${mass*(r*r)/2}" />
+    </macro>
 </robot>
